Commit message: Kamera ide, verte mi.

File: mrvk_description/urdf/robot2.plugins.xacro (robot description, xacro)
@@ -1,5 +1,37 @@
 <?xml version="1.0"?>
 <robot>
-  <!-- hokuyo -->
+ <gazebo reference="camera">
+    <!--material>Gazebo/Green</material-->
+    <sensor type="camera" name="camera1">
+      <update_rate>30.0</update_rate>
+      <camera name="head">
+        <horizontal_fov>1.3962634</horizontal_fov>
+        <image>
+          <width>800</width>
+          <height>800</height>
+          <format>R8G8B8</format>
+        </image>
+        <clip>
+          <near>0.02</near>
+          <far>300</far>
+        </clip>
+      </camera>
+      <plugin name="camera_controller" filename="libgazebo_ros_camera.so">
+        <alwaysOn>true</alwaysOn>
+        <updateRate>0.0</updateRate>
+        <cameraName>camera</cameraName>
+        <imageTopicName>image_raw</imageTopicName>
+        <cameraInfoTopicName>camera_info</cameraInfoTopicName>
+        <frameName>camera_link</frameName>
+        <hackBaseline>0.07</hackBaseline>
+        <distortionK1>0.0</distortionK1>
+        <distortionK2>0.0</distortionK2>
+        <distortionK3>0.0</distortionK3>
+        <distortionT1>0.0</distortionT1>
+        <distortionT2>0.0</distortionT2>
+      </plugin>
+    </sensor>
+  </gazebo>
+  <!-- Lidar hokuyo -->
   <gazebo reference="sensor_laser">
     <sensor type="gpu_ray" name="head_hokuyo_sensor">

File: mrvk_description/urdf/robot2.urdf.xacro (robot description, xacro)
@@ -9,4 +9,5 @@
     <xacro:property name="laser_origin_y" value="0"/>
     <xacro:property name="laser_origin_z" value="0.12"/>
+     <xacro:property name="camera_link" value="0.05" />
     <xacro:macro name="default_inertial" params="mass">
         <inertial>
@@ -126,3 +127,30 @@
     <child link="sensor_laser" />
   </joint>
+  <!-- Camera -->
+  <link name="camera">
+    <collision>
+      <origin xyz="0 0 0" rpy="0 0 0"/>
+      <geometry>
+        <box size="${camera_link} ${camera_link} ${camera_link}"/>
+      </geometry>
+    </collision>
+    <visual>
+      <origin xyz="0 0 0" rpy="0 0 0"/>
+      <geometry>
+        <box size="${camera_link} ${camera_link} ${camera_link}"/>
+      </geometry>
+      <material name="red"/>
+    </visual>
+    <inertial>
+      <mass value="1e-5" />
+      <origin xyz="0 0 0" rpy="0 0 0"/>
+      <inertia ixx="1e-6" ixy="0" ixz="0" iyy="1e-6" iyz="0" izz="1e-6" />
+    </inertial>
+  </link>
+  <joint name="camera_joint" type="fixed">
+    <axis xyz="0 1 0" />
+    <origin xyz="0.3 0 0" rpy="0 0 0"/>
+    <parent link="base_link"/>
+    <child link="camera"/>
+  </joint>
 </robot>
