Commit message: uprava parametrov

File: mrvk_description/urdf/robot2.urdf.xacro (robot description, xacro)
@@ -32,11 +32,11 @@
                 </geometry>
             </collision>
-            <xacro:default_inertial mass="10" />
+            <xacro:default_inertial mass= "${mass}"/>
         </link>
     </xacro:macro>
     <!-- Macro koleso -->
-    <xacro:macro name="wheel" params="prefix radius length joint_xyz">
+    <xacro:macro name="wheel" params="prefix radius length joint_xyz mass">
         <link name="wheel_${prefix}_link">
-            <xacro:default_inertial mass="1"/>
+            <xacro:default_inertial mass="${mass}"/>
             <visual>
                 <origin xyz="0.0 0.0 0.0" rpy="0.0 0.0 0.0"/>
@@ -57,5 +57,5 @@
             <parent link="base_link"/>
             <child link="wheel_${prefix}_link"/>
-            <axis xyz="0 0 1"/>
+            <axis xyz="0 0 -1"/>
         </joint>
         <transmission name="${prefix}_wheel_trans">
@@ -71,5 +71,5 @@
             <mu1 value="200.0"/>
             <mu2 value="100.0"/>
-            <kp value="10000000.0" />
+            <kp value="100000.0" />
             <kd value="1.0" />
             <material>Gazebo/Grey</material>
@@ -78,28 +78,32 @@
     <!--  -->
     <xacro:box_link
+        name="base_link"
         size_x="0.47" size_y="0.315" size_z="0.168"
-        mass="10"
-        name="base_link"
-        material_name="Blue" />
+        mass="30"
+        material_name="Blue"/>
     <xacro:wheel
         prefix="left_front"
         radius="0.115"
         length="0.065"
-        joint_xyz="0.145 0.20 -0.01"/>
+        joint_xyz="0.145 0.20 -0.01"
+        mass = "0.5"/>
     <xacro:wheel
         prefix="left_back"
         radius="0.115"
         length="0.065"
-        joint_xyz="-0.145 0.20 -0.01"/>
+        joint_xyz="-0.145 0.20 -0.01"
+        mass = "0.5"/>
     <xacro:wheel
         prefix="right_front"
         radius="0.115"
         length="0.065"
-        joint_xyz="0.145 -0.20 -0.01"/>
+        joint_xyz="0.145 -0.20 -0.01"
+        mass = "0.5"/>
     <xacro:wheel
         prefix="right_back"
         radius="0.115"
         length="0.065"
-        joint_xyz="-0.145 -0.20 -0.01"/>
+        joint_xyz="-0.145 -0.20 -0.01"
+        mass = "0.5"/>
     <!--gazebo>
         <plugin name="gazebo_ros_control" filename="libgazebo_ros_control.so">
@@ -118,5 +122,5 @@
         <wheelDiameter>0.23</wheelDiameter>
         <robotBaseFrame>base_link</robotBaseFrame>
-        <torque>100</torque>
+        <torque>5</torque>
         <commandTopic>cmd_vel</commandTopic>
         <odometryTopic>odom</odometryTopic>

Commit message: path_detection updated

File: mrvk_description/urdf/robot2.urdf.xacro (robot description, xacro)
@@ -184,5 +184,5 @@
   <joint name="camera_joint" type="fixed">
     <axis xyz="0 1 0" />
-    <origin xyz="0.3 0 0" rpy="0 0 0"/>
+    <origin xyz="0.3 0 0.5" rpy="0 0 0"/>
     <parent link="base_link"/>
     <child link="camera"/>
