Commit message: rozdelenie urdf

File: mrvk_description/urdf/materials.urdf.xacro (robot description, xacro)
@@ -1,19 +1,22 @@
 <?xml version="1.0"?>
-<robot name="mrvk" xmlns:xacro="http://ros.org/wiki/xacro">
-<material name="Black">
-    <color rgba="0.0 0.0 0.0 1.0"/>
-</material>
-<material name="Blue">
-    <color rgba="0.0 0.0 0.8 1.0"/>
-</material>
-<material name="Green">
-    <color rgba="0.0 0.8 0.0 1.0"/>
-</material>
-<material name="Grey">
-    <color rgba="0.2 0.2 0.2 1.0"/>
-</material>
-<material name="White">
-    <color rgba="1.0 1.0 1.0 1.0"/>
-</material>
+<robot name="shoddy" xmlns:xacro="http://ros.org/wiki/xacro">
+    <material name="Black">
+        <color rgba="0.0 0.0 0.0 1.0"/>
+    </material>
+    <material name="Blue">
+        <color rgba="0.0 0.0 0.8 1.0"/>
+    </material>
+    <material name="Green">
+        <color rgba="0.0 0.8 0.0 1.0"/>
+    </material>
+    <material name="Grey">
+        <color rgba="0.5 0.5 0.5 1.0"/>
+    </material>
+    <material name="DarkGrey">
+        <color rgba="0.2 0.2 0.2 1.0"/>
+    </material>
+    <material name="White">
+        <color rgba="1.0 1.0 1.0 1.0"/>
+    </material>
     <material name= "kinect">
         <color rgba="0.2 0.2 0.2 1.0"/>

File: mrvk_description/urdf/robot.urdf.xacro (robot description, xacro)
@@ -1,29 +1,36 @@
 <?xml version="1.0"?>
-<robot xmlns:xacro="http://ros.org/wiki/xacro"
-       xmlns:xi="http://www.w3.org/2001/XInclude"
-       xmlns:gazebo="http://playerstage.sourceforge.net/gazebo/xmlschema/#gz"
-       xmlns:model="http://playerstage.sourceforge.net/gazebo/xmlschema/#model"
-       xmlns:sensor="http://playerstage.sourceforge.net/gazebo/xmlschema/#sensor"
-       xmlns:body="http://playerstage.sourceforge.net/gazebo/xmlschema/#body"
-       xmlns:geom="http://playerstage.sourceforge.net/gazebo/xmlschema/#geom"
-       xmlns:joint="http://playerstage.sourceforge.net/gazebo/xmlschema/#joint"
-       xmlns:interface="http://playerstage.sourceforge.net/gazebo/xmlschema/#interface"
-       xmlns:rendering="http://playerstage.sourceforge.net/gazebo/xmlschema/#rendering"
-       xmlns:renderable="http://playerstage.sourceforge.net/gazebo/xmlschema/#renderable"
-       xmlns:controller="http://playerstage.sourceforge.net/gazebo/xmlschema/#controller"
-       xmlns:physics="http://playerstage.sourceforge.net/gazebo/xmlschema/#physics"
-       name="mrvk" >
-  <!-- common stuff -->
-  <xacro:include filename="$(find mrvk_description)/urdf/materials.urdf.xacro" />
-  <xacro:include filename="$(find mrvk_description)/urdf/common.urdf.xacro" />
-  <xacro:include filename="$(find mrvk_description)/urdf/mrvk.urdf.xacro" />
- <!--  <xacro:include filename="$(find mrvk_description)/urdf/kv01.urdf.xacro" /> -->
-  <!-- Used for fixing robot to Gazebo -->
-  <!--<link name="world"/>-->
-  <!-- arm -->
-  <xacro:mrvk_base parent="world" end_point = "base_end_point">
-     <origin xyz="0 0 0" rpy="0 0 0" />
-  </xacro:mrvk_base>
-  <!--<xacro:kv01_arm parent="base_end_point" end_point = "tool_point">-->
-  <!--</xacro:kv01_arm>-->
+<robot name="shoddy" xmlns:xacro="http://wiki.ros.org/xacro">
+    <xacro:include filename="$(find mrvk_description)/urdf/robot.plugins.xacro"/>
+    <xacro:include filename="$(find mrvk_description)/urdf/materials.urdf.xacro"/>
+    <xacro:include filename="$(find mrvk_description)/urdf/base_macro.urdf.xacro"/>
+    <xacro:include filename="$(find mrvk_description)/urdf/wheel_macro.urdf.xacro"/>
+    <xacro:include filename="$(find mrvk_description)/urdf/camera_macro.urdf.xacro"/>
+    <xacro:include filename="$(find mrvk_description)/urdf/lidar_macro.urdf.xacro"/>
+    <!-- Body -->
+    <xacro:base_macro name="base_link"/>
+    <!-- Wheels -->
+    <xacro:wheel_macro
+        side="left"
+        part="front"
+        origin="0.145 0.20 -0.02"
+        parent="base_link"/>
+    <xacro:wheel_macro
+        side="left"
+        part="rear"
+        origin="-0.145 0.20 -0.02"
+        parent="base_link"/>
+    <xacro:wheel_macro
+        side="right"
+        part="front"
+        origin="0.145 -0.20 -0.02"
+        parent="base_link"/>
+    <xacro:wheel_macro
+        side="right"
+        part="rear"
+        origin="-0.145 -0.20 -0.02"
+        parent="base_link"/>
+    <!-- LIDAR -->
+    <xacro:lidar_macro name="sensor_laser_link" parent="base_link"/>
+    <!-- Camera -->
+    <xacro:camera_macro name="camera_link" parent="base_link"/>
 </robot>
