Commit message: posledna verzia vylepseneho modelu 1.0 :)

File: mrvk_description/urdf/camera_macro.urdf.xacro (robot description, xacro)
@@ -2,42 +2,199 @@
 <robot name="shoddy" xmlns:xacro="http://wiki.ros.org/xacro">
     <xacro:macro name="camera_macro" params="name parent">
-        <!-- Properties -->
-        <!-- Lens -->
-        <xacro:property name="lens_radius" value="0.015"/>
-        <xacro:property name="lens_length" value="0.04"/>
-        <xacro:property name="lens_shift_x" value="${box_size_x/2}"/>
+        <!-- Properties ==================================================== -->
+        <!-- Base -->
+        <!-- Base upper -->
+        <xacro:property name="base_upper_radius" value="0.058"/>
+        <xacro:property name="base_upper_length" value="0.025"/>
+        <xacro:property name="base_upper_x" value="0.16"/>
+        <xacro:property name="base_upper_y" value="0.0"/>
+        <xacro:property name="base_upper_z" value="${0.084 + base_lower_length + base_shift_z}"/>
+        <!-- Base lower -->
+        <xacro:property name="base_lower_radius" value="0.02"/>
+        <xacro:property name="base_lower_length" value="0.041"/>
+        <xacro:property name="base_lower_x" value="${base_upper_x - base_upper_radius + base_lower_radius}"/>
+        <xacro:property name="base_lower_y" value="0.0"/>
+        <xacro:property name="base_lower_z" value="${0.084 + base_lower_length/2}"/>
+        <!-- Base holder -->
+        <xacro:property name="base_holder_radius" value="0.005"/>
+        <xacro:property name="base_holder_length" value="${box_size_y + 0.01}"/>
+        <xacro:property name="base_holder_x" value="${box_x}"/>
+        <xacro:property name="base_holder_y" value="${box_y}"/>
+        <xacro:property name="base_holder_z" value="${box_z}"/>
+        <xacro:property name="base_shift_z" value="${base_upper_length/2}"/>
+        <xacro:property name="pitch" value="${pi/8}"/>
+        <xacro:property name="base_material" value="Grey"/>
+        <!-- Base -->
+        <!-- Holder -->
+        <xacro:property name="C" value="${sqrt(2)}"/>
+        <xacro:property name="holder_lower_width" value="${box_size_x}"/>
+        <xacro:property name="holder_upper_width" value="${box_size_x/2}"/>
+        <xacro:property name="holder_height" value="0.30"/>
+        <xacro:property name="holder_width" value="0.01"/>
+        <xacro:property name="holder_corner_size" value="${1/C*(holder_lower_width - holder_upper_width)}"/>
+        <xacro:property name="holder_x" value="${base_upper_x}"/>
+        <xacro:property name="holder_left_y" value="${-box_size_y/2 - holder_width/2 - 0.005}"/>
+        <xacro:property name="holder_right_y" value="${box_size_y/2 + holder_width/2 + 0.005}"/>
+        <xacro:property name="holder_z" value="${base_upper_z + base_upper_length/2}"/>
+        <xacro:property name="holder_material" value="DarkGrey"/>
+        <!-- Holder -->
+        <!-- Box -->
+        <xacro:property name="box_size_x" value="0.07"/>
+        <xacro:property name="box_size_y" value="0.06"/>
+        <xacro:property name="box_size_z" value="0.06"/>
+        <xacro:property name="box_x" value="${base_upper_x}"/>
+        <xacro:property name="box_y" value="${base_upper_y}"/>
+        <xacro:property name="box_z" value="${base_upper_z + base_shift_z + holder_height - box_size_z/2}"/>
+        <xacro:property name="box_material" value="DarkGrey"/>
+        <!-- Box -->
+        <!-- Lens -->
+        <xacro:property name="lens_radius" value="0.025"/>
+        <xacro:property name="lens_length" value="0.005"/>
+        <xacro:property name="lens_x" value="${box_x + lens_shift_x*cos(pitch)}"/>
+        <xacro:property name="lens_y" value="${box_y}"/>
+        <xacro:property name="lens_z" value="${box_z - lens_shift_x*sin(pitch)}"/>
+        <xacro:property name="lens_shift_x" value="${box_size_x/2 + lens_length/2}"/>
         <xacro:property name="lens_material" value="Black"/>
-        <!-- Box -->
-        <xacro:property name="box_size_x" value="0.07"/>
-        <xacro:property name="box_size_y" value="0.05"/>
-        <xacro:property name="box_size_z" value="0.05"/>
-        <xacro:property name="box_material" value="DarkGrey"/>
-        <!-- Base -->
-        <xacro:property name="base_radius" value="0.01"/>
-        <xacro:property name="base_length" value="0.28"/>
-        <xacro:property name="origin_x" value="0.1"/>
-        <xacro:property name="origin_y" value="0.0"/>
-        <xacro:property name="origin_z" value="${0.084 + base_shift_z}"/>
-        <xacro:property name="base_shift_z" value="${base_length/2}"/>
-        <xacro:property name="pitch" value="${pi/10}"/>
-        <xacro:property name="base_material" value="Grey"/>
-        <!-- Links -->
-        <!-- Lens -->
+        <!-- Lens -->
+        <!-- ==================================================== Properties -->
+        <!-- Macros ======================================================== -->
+        <!-- Base -->
+        <xacro:macro name="base_macro" params="name radius length x y z rpy parent">
+            <link name="${name}_link">
+                <visual>
+                    <origin xyz="0 0 0" rpy="0 0 0"/>
+                    <geometry>
+                        <cylinder radius="${radius}" length="${length}"/>
+                    </geometry>
+                    <material name="${base_material}"/>
+                </visual>
+                <collision>
+                    <origin xyz="0 0 0" rpy="0 0 0"/>
+                    <geometry>
+                        <cylinder radius="${radius}" length="${length}"/>
+                    </geometry>
+                </collision>
+                <inertial>
+                    <origin xyz="0 0 0" rpy="0 0 0"/>
+                    <mass value="0.0"/>
+                    <inertia ixx="0.0" ixy="0.0" ixz="0.0" iyy="0.0" iyz="0.0" izz="0.0"/>
+                </inertial>
+            </link>
+            <joint name="${name}_joint" type="fixed">
+                <origin xyz="${x} ${y} ${z}" rpy="${rpy}"/>
+                <parent link="${parent}"/>
+                <child link="${name}_link"/>
+            </joint>
+            <gazebo reference="${name}_link">
+                <material>Gazebo/Grey</material>
+            </gazebo>
+        </xacro:macro>
+        <!-- Base -->
+        <!-- Holder -->
+        <xacro:macro name="holder_macro" params="name x y z parent">
+            <xacro:macro name="box_macro" params="name size xyz rpy parent">
+                <link name="${name}_link">
+                    <visual>
+                        <origin xyz="0 0 0" rpy="0 0 0"/>
+                        <geometry>
+                            <box size="${size}"/>
+                        </geometry>
+                        <material name="${holder_material}"/>
+                    </visual>
+                    <collision>
+                        <origin xyz="0 0 0" rpy="0 0 0"/>
+                        <geometry>
+                            <box size="${size}"/>
+                        </geometry>
+                    </collision>
+                    <inertial>
+                        <origin xyz="0 0 0" rpy="0 0 0"/>
+                        <mass value="0.0"/>
+                        <inertia ixx="0.0" ixy="0.0" ixz="0.0" iyy="0.0" iyz="0.0" izz="0.0"/>
+                    </inertial>
+                </link>
+                <joint name="${name}_joint" type="fixed">
+                    <origin xyz="${xyz}"
+                            rpy="${rpy}"/>
+                    <parent link="${parent}"/>
+                    <child link="${name}_link"/>
+                </joint>
+                <gazebo reference="${name}_link">
+                    <material>Gazebo/FlatBlack</material>
+                </gazebo>
+            </xacro:macro>
+            <xacro:box_macro name="${name}_1"
+                             size="${holder_lower_width} ${holder_width} ${holder_height - C/2*holder_corner_size}"
+                             xyz="${x} ${y} ${z + (holder_height - C/2*holder_corner_size)/2}"
+                             rpy="0.0 0.0 0.0"
+                             parent="${parent}"/>
+            <xacro:box_macro name="${name}_2"
+                             size="${holder_upper_width} ${holder_width} ${holder_height}"
+                             xyz="${x} ${y} ${z + holder_height/2}"
+                             rpy="0.0 0.0 0.0"
+                             parent="${parent}"/>
+            <xacro:box_macro name="${name}_3"
+                             size="${holder_corner_size} ${holder_width} ${holder_corner_size} "
+                             xyz="${x - holder_upper_width/2} ${y} ${z + (holder_height - C/2*holder_corner_size)}"
+                             rpy="0.0 ${pi/4} 0.0"
+                             parent="${parent}"/>
+            <xacro:box_macro name="${name}_4"
+                             size="${holder_corner_size} ${holder_width} ${holder_corner_size} "
+                             xyz="${x + holder_upper_width/2} ${y} ${z + (holder_height - C/2*holder_corner_size)}"
+                             rpy="0.0 ${pi/4} 0.0"
+                             parent="${parent}"/>
+        </xacro:macro>
+        <!-- Holder -->
+        <!-- Box -->
+        <xacro:macro name="box_macro" params="name size xyz rpy parent">
+            <link name="${name}_link">
+                <visual>
+                    <origin xyz="0 0 0" rpy="0 0 0"/>
+                    <geometry>
+                        <box size="${size}"/>
+                    </geometry>
+                    <material name="${box_material}"/>
+                </visual>
+                <collision>
+                    <origin xyz="0 0 0" rpy="0 0 0"/>
+                    <geometry>
+                        <box size="${size}"/>
+                    </geometry>
+                </collision>
+                <inertial>
+                    <origin xyz="0 0 0" rpy="0 0 0"/>
+                    <mass value="0.0"/>
+                    <inertia ixx="0.0" ixy="0.0" ixz="0.0" iyy="0.0" iyz="0.0" izz="0.0"/>
+                </inertial>
+            </link>
+            <joint name="${name}_joint" type="fixed">
+                <origin xyz="${xyz}"
+                        rpy="${rpy}"/>
+                <parent link="${parent}"/>
+                <child link="${name}_link"/>
+            </joint>
+            <gazebo reference="${name}_link">
+                <material>Gazebo/FlatBlack</material>
+            </gazebo>
+        </xacro:macro>
+        <!-- Box -->
+        <!-- Lens -->
+        <xacro:macro name="lens_macro" params="name radius length xyz rpy parent">
         <link name="${name}">
             <visual>
-                <origin xyz="${lens_shift_x} 0 0" rpy="0 ${pi/2} 0"/>
+                <origin xyz="0.0 0.0 0.0" rpy="0 ${pi/2} 0"/>
                 <geometry>
-                    <cylinder radius="${lens_radius}" length="${lens_length}"/>
+                    <cylinder radius="${radius}" length="${length}"/>
                 </geometry>
                 <material name="${lens_material}"/>
             </visual>
             <collision>
+                <origin xyz="0.0 0.0 0.0" rpy="0 ${pi/2} 0"/>
                 <geometry>
-                    <cylinder radius="${lens_radius}" length="${lens_length}"/>
+                    <cylinder radius="${radius}" length="${length}"/>
                 </geometry>
-                <origin xyz="${lens_shift_x} 0 0" rpy="0 ${pi/2} 0"/>
             </collision>
             <inertial>
-                <origin xyz="${lens_shift_x} 0 0" rpy="0 ${pi/2} 0"/>
+                <origin xyz="0.0 0.0 0.0" rpy="0 ${pi/2} 0"/>
                 <mass value="0.0"/>
                 <inertia ixx="0.0" ixy="0.0" ixz="0.0" iyy="0.0" iyz="0.0" izz="0.0"/>
@@ -45,6 +202,6 @@
         </link>
         <joint name="camera_lens_joint" type="fixed">
-            <origin xyz="${origin_x} ${origin_y} ${origin_z + base_shift_z}"
-                    rpy="0 ${pitch} 0"/>
+            <origin xyz="${xyz}"
+                    rpy="${rpy}"/>
             <parent link="${parent}"/>
             <child link="${name}"/>
@@ -53,64 +210,54 @@
             <material>Gazebo/Black</material>
         </gazebo>
-        <!-- Box -->
-        <link name="camera_box_link">
-            <visual>
-                <origin xyz="0 0 0" rpy="0 0 0"/>
-                <geometry>
-                    <box size="${box_size_x} ${box_size_y} ${box_size_z}"/>
-                    <!-- <mesh filename="package://mrvk_description/meshes/camera/model.dae" scale="0.5 0.5 0.5"/> -->
-                </geometry>
-                <material name="${box_material}"/>
-            </visual>
-            <collision>
-                <origin xyz="0 0 0" rpy="0 0 0"/>
-                <geometry>
-                    <box size="${box_size_x} ${box_size_y} ${box_size_z}"/>
-                </geometry>
-            </collision>
-            <inertial>
-                <origin xyz="0 0 0" rpy="0 0 0"/>
-                <mass value="0.0"/>
-                <inertia ixx="0.0" ixy="0.0" ixz="0.0" iyy="0.0" iyz="0.0" izz="0.0"/>
-            </inertial>
-        </link>
-        <joint name="camera_box_joint" type="fixed">
-            <origin xyz="${origin_x} ${origin_y} ${origin_z + base_shift_z}"
-                    rpy="0.0 ${pitch} 0.0"/>
-            <parent link="${parent}"/>
-            <child link="camera_box_link"/>
-        </joint>
-        <gazebo reference="camera_box_link">
-            <material>Gazebo/DarkGrey</material>
-        </gazebo>
-        <!-- Base -->
-        <link name="camera_base_link">
-            <visual>
-                <origin xyz="0 0 0" rpy="0 0 0"/>
-                <geometry>
-                    <cylinder radius="${base_radius}" length="${base_length}"/>
-                </geometry>
-                <material name="${base_material}"/>
-            </visual>
-            <collision>
-                <origin xyz="0 0 0" rpy="0 0 0"/>
-                <geometry>
-                    <cylinder radius="${base_radius}" length="${base_length}"/>
-                </geometry>
-            </collision>
-            <inertial>
-                <origin xyz="0 0 0" rpy="0 0 0"/>
-                <mass value="0.0"/>
-                <inertia ixx="0.0" ixy="0.0" ixz="0.0" iyy="0.0" iyz="0.0" izz="0.0"/>
-            </inertial>
-        </link>
-        <joint name="camera_base_joint" type="fixed">
-            <origin xyz="${origin_x} ${origin_y} ${origin_z}" rpy="0 0 0"/>
-            <parent link="${parent}"/>
-            <child link="camera_base_link"/>
-        </joint>
-        <gazebo reference="camera_base_link">
-            <material>Gazebo/Grey</material>
-        </gazebo>
+        </xacro:macro>
+        <!-- Lens -->
+        <!-- ======================================================== Macros -->
+        <!-- Links ========================================================= -->
+        <xacro:base_macro name="camera_base_upper"
+                          radius="${base_upper_radius}"
+                          length="${base_upper_length}"
+                          x="${base_upper_x}"
+                          y="${base_upper_y}"
+                          z="${base_upper_z}"
+                          rpy="0.0 0.0 0.0"
+                          parent="${parent}"/>
+        <xacro:base_macro name="camera_base_lower"
+                          radius="${base_lower_radius}"
+                          length="${base_lower_length}"
+                          x="${base_lower_x}"
+                          y="${base_lower_y}"
+                          z="${base_lower_z}"
+                          rpy="0.0 0.0 0.0"
+                          parent="${parent}"/>
+        <xacro:base_macro name="camera_base_holder"
+                          radius="${base_holder_radius}"
+                          length="${base_holder_length}"
+                          x="${base_holder_x}"
+                          y="${base_holder_y}"
+                          z="${base_holder_z}"
+                          rpy="${pi/2} 0.0 0.0"
+                          parent="${parent}"/>
+        <xacro:holder_macro name="camera_holder_left"
+                            x="${holder_x}"
+                            y="${holder_left_y}"
+                            z="${holder_z}"
+                            parent="${parent}"/>
+        <xacro:holder_macro name="camera_holder_right"
+                            x="${holder_x}"
+                            y="${holder_right_y}"
+                            z="${holder_z}"
+                            parent="${parent}"/>
+        <xacro:box_macro name="camera_box"
+                         size="${box_size_x} ${box_size_y} ${box_size_z}"
+                         xyz="${box_x} ${box_y} ${box_z}"
+                         rpy= "0.0 ${pitch} 0.0"
+                         parent="${parent}"/>
+        <xacro:lens_macro name="${name}"
+                          radius="${lens_radius}"
+                          length="${lens_length}"
+                          xyz="${lens_x} ${lens_y} ${lens_z}"
+                          rpy="0.0 ${pitch} 0.0"
+                          parent="${parent}"/>
+        <!-- ========================================================= Links -->
     </xacro:macro>
 </robot>

File: mrvk_description/urdf/lidar_macro.urdf.xacro (robot description, xacro)
@@ -9,5 +9,5 @@
         <xacro:property name="origin_x" value="0.20"/>
         <xacro:property name="origin_y" value="0.0"/>
-        <xacro:property name="origin_z" value="0.12"/>
+        <xacro:property name="origin_z" value="0.09"/>
         <!-- Link -->
         <link name="${name}">

File: mrvk_description/urdf/robot.plugins.xacro (robot description, xacro)
@@ -6,5 +6,5 @@
             <updateRate>50</updateRate>
             <alwaysOn>1</alwaysOn>
-            <robotNamespace>test_robot</robotNamespace>
+            <robotNamespace>shoddy</robotNamespace>
             <leftFrontJoint>wheel_left_front_to_base_joint</leftFrontJoint>
             <leftRearJoint>wheel_left_rear_to_base_joint</leftRearJoint>
@@ -29,5 +29,5 @@
         </plugin>
     </gazebo>
-    <!-- Hokuyo UTM-30LX Laser Range Finder-->
+    <!-- Hokuyo URG-04LX Laser Range Finder-->
     <gazebo reference="sensor_laser_link">
         <sensor type="gpu_ray" name="head_hokuyo_sensor">
@@ -37,7 +37,7 @@
             <ray>
                 <scan>
-                    <horizontal>
-                        <samples>720</samples>
-                        <!--resolution>0.5</resolution-->
+                    <horizontal> -->
+                        <!-- <resolution>0.36</resolution>                         -->
+                        <samples>1000</samples>
                         <min_angle>-3.14159</min_angle>
                         <max_angle>3.14159</max_angle>

File: mrvk_description/urdf/robot.urdf.xacro (robot description, xacro)
@@ -5,6 +5,7 @@
     <xacro:include filename="$(find mrvk_description)/urdf/base_macro.urdf.xacro"/>
     <xacro:include filename="$(find mrvk_description)/urdf/wheel_macro.urdf.xacro"/>
+    <xacro:include filename="$(find mrvk_description)/urdf/lidar_macro.urdf.xacro"/>
     <xacro:include filename="$(find mrvk_description)/urdf/camera_macro.urdf.xacro"/>
-    <xacro:include filename="$(find mrvk_description)/urdf/lidar_macro.urdf.xacro"/>
+    <xacro:include filename="$(find mrvk_description)/urdf/ultrasonic_sensor_macro.urdf.xacro"/>
     <!-- Body -->
     <xacro:base_macro name="base_link"/>
@@ -13,20 +14,20 @@
         side="left"
         part="front"
-        origin="0.145 0.20 -0.02"
+        origin="0.14 0.20 -0.05"
         parent="base_link"/>
     <xacro:wheel_macro
         side="left"
         part="rear"
-        origin="-0.145 0.20 -0.02"
+        origin="-0.14 0.20 -0.05"
         parent="base_link"/>
     <xacro:wheel_macro
         side="right"
         part="front"
-        origin="0.145 -0.20 -0.02"
+        origin="0.14 -0.20 -0.05"
         parent="base_link"/>
     <xacro:wheel_macro
         side="right"
         part="rear"
-        origin="-0.145 -0.20 -0.02"
+        origin="-0.14 -0.20 -0.05"
         parent="base_link"/>
     <!-- LIDAR -->
@@ -34,3 +35,10 @@
     <!-- Camera -->
     <xacro:camera_macro name="camera_link" parent="base_link"/>
+    <!-- Ultrasonic sensors -->
+    <xacro:ultrasonic_sensor_macro name="ultrasonic_sensor_front_left_link" xyz="0.235 ${-0.315/2*0.7} 0.05" parent="base_link"/>
+    <xacro:ultrasonic_sensor_macro name="ultrasonic_sensor_front_middle_link" xyz="0.235 0.0 0.05" parent="base_link"/>
+    <xacro:ultrasonic_sensor_macro name="ultrasonic_sensor_front_right_link" xyz="0.235 ${0.315/2*0.7} 0.05" parent="base_link"/>
+    <xacro:ultrasonic_sensor_macro name="ultrasonic_sensor_rear_left_link" xyz="-0.235 ${-0.315/2*0.7} 0.05" parent="base_link"/>
+    <xacro:ultrasonic_sensor_macro name="ultrasonic_sensor_rear_middle_link" xyz="-0.235 0.0 0.05" parent="base_link"/>
+    <xacro:ultrasonic_sensor_macro name="ultrasonic_sensor_rear_right_link" xyz="-0.235 ${0.315/2*0.7} 0.05" parent="base_link"/>
 </robot>

File: mrvk_description/urdf/wheel_macro.urdf.xacro (robot description, xacro)
@@ -11,5 +11,5 @@
         <link name="wheel_${side}_${part}_link">
             <visual>
-                <origin xyz="0.0 0.0 0.0" rpy="0.0 0.0 0.0"/>
+                <origin xyz="0.0 0.0 0.0" rpy="${pi/2*0.0} 0.0 0.0"/>
                 <geometry>
                     <!-- <cylinder radius="${radius}" length="${length}"/> -->
@@ -46,11 +46,4 @@
             </joint>
         </transmission>
-        <!-- <gazebo reference="${side}_${part}_wheel">
-            <mu1 value="200.0"/>
-            <mu2 value="100.0"/>
-            <kp value="100000.0"/>
-            <kd value="1.0" />
-            <material>Gazebo/FlatBlack</material>
-        </gazebo> -->
         <gazebo reference="wheel_${side}_${part}_link">
             <mu1 value="1.0"/>
