Commit message: add IMU

File: mrvk_description/urdf/base_macro.urdf.xacro (robot description, xacro)
@@ -252,3 +252,28 @@
         <!-- ======================================================= Links -->
     </xacro:macro>
+    <joint name="imu_joint" type="fixed">
+        <axis xyz="1 0 0"/> <!-- 0 1 0 -->
+        <origin xyz="0 0 0.19"/>
+        <parent link="base_link"/>
+        <child link="imu_link"/>
+    </joint>
+    <link name="imu_link">
+      <inertial>
+        <mass value="0.001"/>
+        <origin rpy="0 0 0" xyz="0 0 0"/>
+        <inertia ixx="0.0001" ixy="0" ixz="0" iyy="0.000001" iyz="0" izz="0.0001"/>
+      </inertial>
+      <visual>
+        <origin rpy="0 0 0" xyz="0 0 0"/>
+        <geometry>
+          <box size="0.001 0.001 0.001"/>
+        </geometry>
+      </visual>
+      <collision>
+        <origin rpy="0 0 0" xyz="0 0 0"/>
+        <geometry>
+          <box size=".001 .001 .001"/>
+        </geometry>
+      </collision>
+    </link>
 </robot>

File: mrvk_description/urdf/robot.plugins.xacro (robot description, xacro)
@@ -97,3 +97,14 @@
         </sensor>
     </gazebo>
+    <gazebo>
+        <plugin name="imu_plugin" filename="libgazebo_ros_imu.so">
+            <alwaysOn>true</alwaysOn>
+            <bodyName>imu_link</bodyName>
+            <topicName>imu_data</topicName>
+            <gaussianNoise>2.89e-08</gaussianNoise>
+            <updateRate>20.0</updateRate>
+            <xyzOffsets>0 0 0</xyzOffsets>
+            <rpyOffsets>0 0 0</rpyOffsets>
+        </plugin>
+    </gazebo>
 </robot>

Commit message: Add files via upload

File: mrvk_description/urdf/base_macro.urdf.xacro (robot description, xacro)
@@ -1,4 +1,21 @@
 <?xml version="1.0"?>
 <robot name="shoddy" xmlns:xacro="http://wiki.ros.org/xacro">
+    <!-- Global properties ================================================= -->
+    <!-- Shaft -->
+    <xacro:property name="shaft_radius" value="0.015"/>
+    <xacro:property name="shaft_length" value="0.38"/>
+    <xacro:property name="shaft_front_x" value="0.14"/>
+    <xacro:property name="shaft_front_y" value="0.0"/>
+    <xacro:property name="shaft_front_z" value="-0.05"/>
+    <xacro:property name="shaft_rear_x" value="-0.14"/>
+    <xacro:property name="shaft_rear_y" value="0.0"/>
+    <xacro:property name="shaft_rear_z" value="-0.05"/>
+    <!-- Shaft -->
+    <!-- Base -->
+    <xacro:property name="base_size_x" value="0.47"/>
+    <xacro:property name="base_size_y" value="0.315"/>
+    <xacro:property name="base_size_z" value="0.168"/>
+    <!-- Base -->
+    <!-- ================================================= Global properties -->
     <xacro:macro name="base_macro" params="name">
         <!-- Properties ==================================================== -->
@@ -29,8 +46,4 @@
         <!-- Accessory -->
         <!-- Shaft -->
-        <xacro:property name="shaft_radius" value="0.015"/>
-        <xacro:property name="shaft_length" value="0.38"/>
-        <xacro:property name="shaft_front_xyz" value="0.145 0.0 -0.05"/>
-        <xacro:property name="shaft_rear_xyz" value="-0.145 0.0 -0.05"/>
         <xacro:property name="shaft_material" value="Grey"/>
         <!-- Shaft -->
@@ -44,30 +57,4 @@
         <!-- ==================================================== Properties -->
         <!-- Macros ======================================================== -->
-        <!-- Shaft -->
-        <xacro:macro name="shaft_macro" params="name xyz parent">
-            <link name="${name}_link">
-                <visual>
-                    <origin xyz="0.0 0.0 0.0" rpy="${pi/2} 0.0 0.0"/>
-                    <geometry>
-                        <cylinder radius="${shaft_radius}" length="${shaft_length}"/>
-                    </geometry>
-                    <material name="${shaft_material}"/>
-                </visual>
-                <inertial>
-                    <origin xyz="0.0 0.0 0.0" rpy="${pi/2} 0.0 0.0"/>
-                    <mass value="0.0"/>
-                    <inertia ixx="0.0" ixy="0.0" ixz="0.0" iyy="0.0" iyz="0.0" izz="0.0"/>
-                </inertial>
-            </link>
-            <joint name="${name}_joint" type="fixed">
-                <origin xyz="${xyz}" rpy="0.0 0.0 0.0"/>
-                <parent link="${parent}"/>
-                <child link="${name}_link"/>
-            </joint>
-            <gazebo reference="${name}_link">
-                <material>Gazebo/Grey</material>
-            </gazebo>
-        </xacro:macro>
-        <!-- Shaft -->
         <!-- Bumper -->
         <!-- Holder -->
@@ -168,4 +155,30 @@
         </xacro:macro>
         <!-- Accessory -->
+        <!-- Shaft -->
+        <xacro:macro name="shaft_macro" params="name xyz parent">
+            <link name="${name}_link">
+                <visual>
+                    <origin xyz="0.0 0.0 0.0" rpy="${pi/2} 0.0 0.0"/>
+                    <geometry>
+                        <cylinder radius="${shaft_radius}" length="${shaft_length}"/>
+                    </geometry>
+                    <material name="${shaft_material}"/>
+                </visual>
+                <inertial>
+                    <origin xyz="0.0 0.0 0.0" rpy="${pi/2} 0.0 0.0"/>
+                    <mass value="0.0"/>
+                    <inertia ixx="0.0" ixy="0.0" ixz="0.0" iyy="0.0" iyz="0.0" izz="0.0"/>
+                </inertial>
+            </link>
+            <joint name="${name}_joint" type="fixed">
+                <origin xyz="${xyz}" rpy="0.0 0.0 0.0"/>
+                <parent link="${parent}"/>
+                <child link="${name}_link"/>
+            </joint>
+            <gazebo reference="${name}_link">
+                <material>Gazebo/Grey</material>
+            </gazebo>
+        </xacro:macro>
+        <!-- Shaft -->
         <!-- Base -->
         <xacro:macro name="base_macro" params="name">
@@ -202,8 +215,8 @@
         <!-- Shafts -->
         <xacro:shaft_macro name="shaft_front"
-                           xyz="${shaft_front_xyz}"
+                           xyz="${shaft_front_x} ${shaft_front_y} ${shaft_front_z}"
                            parent="${name}"/>
         <xacro:shaft_macro name="shaft_rear"
-                           xyz="${shaft_rear_xyz}"
+                           xyz="${shaft_rear_x} ${shaft_rear_y} ${shaft_rear_z}"
                            parent="${name}"/>
         <!-- Shafts -->
@@ -252,28 +265,3 @@
         <!-- ======================================================= Links -->
     </xacro:macro>
-    <joint name="imu_joint" type="fixed">
-        <axis xyz="1 0 0"/> <!-- 0 1 0 -->
-        <origin xyz="0 0 0.19"/>
-        <parent link="base_link"/>
-        <child link="imu_link"/>
-    </joint>
-    <link name="imu_link">
-      <inertial>
-        <mass value="0.001"/>
-        <origin rpy="0 0 0" xyz="0 0 0"/>
-        <inertia ixx="0.0001" ixy="0" ixz="0" iyy="0.000001" iyz="0" izz="0.0001"/>
-      </inertial>
-      <visual>
-        <origin rpy="0 0 0" xyz="0 0 0"/>
-        <geometry>
-          <box size="0.001 0.001 0.001"/>
-        </geometry>
-      </visual>
-      <collision>
-        <origin rpy="0 0 0" xyz="0 0 0"/>
-        <geometry>
-          <box size=".001 .001 .001"/>
-        </geometry>
-      </collision>
-    </link>
 </robot>

File: mrvk_description/urdf/camera_macro.urdf.xacro (robot description, xacro)
@@ -9,5 +9,5 @@
         <xacro:property name="base_upper_x" value="0.16"/>
         <xacro:property name="base_upper_y" value="0.0"/>
-        <xacro:property name="base_upper_z" value="${0.084 + base_lower_length + base_shift_z}"/>
+        <xacro:property name="base_upper_z" value="${base_size_z/2 + base_lower_length + base_upper_length/2}"/>
         <!-- Base lower -->
         <xacro:property name="base_lower_radius" value="0.02"/>
@@ -15,5 +15,5 @@
         <xacro:property name="base_lower_x" value="${base_upper_x - base_upper_radius + base_lower_radius}"/>
         <xacro:property name="base_lower_y" value="0.0"/>
-        <xacro:property name="base_lower_z" value="${0.084 + base_lower_length/2}"/>
+        <xacro:property name="base_lower_z" value="${base_size_z/2 + base_lower_length/2}"/>
         <!-- Base holder -->
         <xacro:property name="base_holder_radius" value="0.005"/>
@@ -22,5 +22,4 @@
         <xacro:property name="base_holder_y" value="${box_y}"/>
         <xacro:property name="base_holder_z" value="${box_z}"/>
-        <xacro:property name="base_shift_z" value="${base_upper_length/2}"/>
         <xacro:property name="pitch" value="${pi/8}"/>
         <xacro:property name="base_material" value="Grey"/>
@@ -45,5 +44,5 @@
         <xacro:property name="box_x" value="${base_upper_x}"/>
         <xacro:property name="box_y" value="${base_upper_y}"/>
-        <xacro:property name="box_z" value="${base_upper_z + base_shift_z + holder_height - box_size_z/2}"/>
+        <xacro:property name="box_z" value="${base_upper_z + base_upper_length/2 + holder_height - box_size_z/2}"/>
         <xacro:property name="box_material" value="DarkGrey"/>
         <!-- Box -->

File: mrvk_description/urdf/robot.plugins.xacro (robot description, xacro)
@@ -14,6 +14,6 @@
             <wheelDiameter>0.23</wheelDiameter>
             <robotBaseFrame>base_link</robotBaseFrame>
-            <wheel_accel>1</wheel_accel>
-            <torque>8</torque>
+            <wheel_accel>2</wheel_accel>
+            <torque>10</torque>
             <commandTopic>cmd_vel</commandTopic>
             <odometryTopic>odom</odometryTopic>
@@ -29,4 +29,16 @@
         </plugin>
     </gazebo>
+    <!-- IMU -->
+    <gazebo>
+        <plugin name="imu_plugin" filename="libgazebo_ros_imu.so">
+            <alwaysOn>true</alwaysOn>
+            <bodyName>imu_link</bodyName>
+            <topicName>imu_data</topicName>
+            <gaussianNoise>2.89e-08</gaussianNoise>
+            <updateRate>20.0</updateRate>
+            <xyzOffsets>0 0 0</xyzOffsets>
+            <rpyOffsets>0 0 0</rpyOffsets>
+        </plugin>
+    </gazebo>
     <!-- Hokuyo URG-04LX Laser Range Finder-->
     <gazebo reference="sensor_laser_link">
@@ -37,6 +49,6 @@
             <ray>
                 <scan>
-                    <horizontal> -->
-                        <!-- <resolution>0.36</resolution>                         -->
+                    <horizontal>
+                        <!-- <resolution>0.36</resolution> -->
                         <samples>1000</samples>
                         <min_angle>-3.14159</min_angle>
@@ -97,14 +109,3 @@
         </sensor>
     </gazebo>
-    <gazebo>
-        <plugin name="imu_plugin" filename="libgazebo_ros_imu.so">
-            <alwaysOn>true</alwaysOn>
-            <bodyName>imu_link</bodyName>
-            <topicName>imu_data</topicName>
-            <gaussianNoise>2.89e-08</gaussianNoise>
-            <updateRate>20.0</updateRate>
-            <xyzOffsets>0 0 0</xyzOffsets>
-            <rpyOffsets>0 0 0</rpyOffsets>
-        </plugin>
-    </gazebo>
 </robot>

File: mrvk_description/urdf/robot.urdf.xacro (robot description, xacro)
@@ -5,4 +5,5 @@
     <xacro:include filename="$(find mrvk_description)/urdf/base_macro.urdf.xacro"/>
     <xacro:include filename="$(find mrvk_description)/urdf/wheel_macro.urdf.xacro"/>
+    <xacro:include filename="$(find mrvk_description)/urdf/imu_macro.urdf.xacro"/>
     <xacro:include filename="$(find mrvk_description)/urdf/lidar_macro.urdf.xacro"/>
     <xacro:include filename="$(find mrvk_description)/urdf/camera_macro.urdf.xacro"/>
@@ -14,21 +15,23 @@
         side="left"
         part="front"
-        origin="0.14 0.20 -0.05"
+        xyz="${shaft_front_x} 0.2 ${shaft_front_z}"
         parent="base_link"/>
     <xacro:wheel_macro
         side="left"
         part="rear"
-        origin="-0.14 0.20 -0.05"
+        xyz="${shaft_rear_x} 0.2 ${shaft_rear_z}"
         parent="base_link"/>
     <xacro:wheel_macro
         side="right"
         part="front"
-        origin="0.14 -0.20 -0.05"
+        xyz="${shaft_front_x} -0.2 ${shaft_front_z}"
         parent="base_link"/>
     <xacro:wheel_macro
         side="right"
         part="rear"
-        origin="-0.14 -0.20 -0.05"
+        xyz="${shaft_rear_x} -0.2 ${shaft_rear_z}"
         parent="base_link"/>
+    <!-- IMU -->
+    <xacro:imu_macro name="imu_link" xyz="0.0 0.0 0.0" parent="base_link"/>
     <!-- LIDAR -->
     <xacro:lidar_macro name="sensor_laser_link" parent="base_link"/>
@@ -36,9 +39,27 @@
     <xacro:camera_macro name="camera_link" parent="base_link"/>
     <!-- Ultrasonic sensors -->
-    <xacro:ultrasonic_sensor_macro name="ultrasonic_sensor_front_left_link" xyz="0.235 ${-0.315/2*0.7} 0.05" parent="base_link"/>
-    <xacro:ultrasonic_sensor_macro name="ultrasonic_sensor_front_middle_link" xyz="0.235 0.0 0.05" parent="base_link"/>
-    <xacro:ultrasonic_sensor_macro name="ultrasonic_sensor_front_right_link" xyz="0.235 ${0.315/2*0.7} 0.05" parent="base_link"/>
-    <xacro:ultrasonic_sensor_macro name="ultrasonic_sensor_rear_left_link" xyz="-0.235 ${-0.315/2*0.7} 0.05" parent="base_link"/>
-    <xacro:ultrasonic_sensor_macro name="ultrasonic_sensor_rear_middle_link" xyz="-0.235 0.0 0.05" parent="base_link"/>
-    <xacro:ultrasonic_sensor_macro name="ultrasonic_sensor_rear_right_link" xyz="-0.235 ${0.315/2*0.7} 0.05" parent="base_link"/>
+    <xacro:ultrasonic_sensor_macro
+        name="ultrasonic_sensor_front_left_link"
+        xyz="${base_size_x/2} ${-base_size_y/2*0.7} 0.05"
+        parent="base_link"/>
+    <xacro:ultrasonic_sensor_macro
+        name="ultrasonic_sensor_front_middle_link"
+        xyz="${base_size_x/2} 0.0 0.05"
+        parent="base_link"/>
+    <xacro:ultrasonic_sensor_macro
+        name="ultrasonic_sensor_front_right_link"
+        xyz="${base_size_x/2} ${base_size_y/2*0.7} 0.05"
+        parent="base_link"/>
+    <xacro:ultrasonic_sensor_macro
+        name="ultrasonic_sensor_rear_left_link"
+        xyz="${-base_size_x/2} ${-base_size_y/2*0.7} 0.05"
+        parent="base_link"/>
+    <xacro:ultrasonic_sensor_macro
+        name="ultrasonic_sensor_rear_middle_link"
+        xyz="${-base_size_x/2} 0.0 0.05"
+        parent="base_link"/>
+    <xacro:ultrasonic_sensor_macro
+        name="ultrasonic_sensor_rear_right_link"
+        xyz="${-base_size_x/2} ${base_size_y/2*0.7} 0.05"
+        parent="base_link"/>
 </robot>

File: mrvk_description/urdf/wheel_macro.urdf.xacro (robot description, xacro)
@@ -1,6 +1,6 @@
 <?xml version="1.0"?>
 <robot name="shoddy" xmlns:xacro="http://wiki.ros.org/xacro">
-    <xacro:macro name="wheel_macro" params="side part origin parent">
-        <!-- Properties -->
+    <xacro:macro name="wheel_macro" params="side part xyz parent">
+        <!-- Properties ==================================================== -->
         <xacro:property name="radius" value="0.115"/>
         <xacro:property name="length" value="0.065"/>
@@ -8,10 +8,10 @@
         <xacro:property name="Cr" value="${0.001/0.033}"/>
         <xacro:property name="Cl" value="${0.001/0.018}"/>
-        <!-- Link -->
+        <!-- ==================================================== Properties -->
+        <!-- Link ========================================================== -->
         <link name="wheel_${side}_${part}_link">
             <visual>
                 <origin xyz="0.0 0.0 0.0" rpy="${pi/2*0.0} 0.0 0.0"/>
                 <geometry>
-                    <!-- <cylinder radius="${radius}" length="${length}"/> -->
                     <mesh filename="package://mrvk_description/meshes/wheels/${side}_tire.stl"
                           scale="${Cr*radius} ${Cl*length} ${Cr*radius}"/>
@@ -32,6 +32,6 @@
         </link>
         <joint name="wheel_${side}_${part}_to_base_joint" type="continuous">
-            <axis xyz="0 1 0"/>
-            <origin xyz="${origin}" rpy="0.0 0.0 0.0"/>
+            <axis xyz="0.0 1.0 0.0"/>
+            <origin xyz="${xyz}" rpy="0.0 0.0 0.0"/>
             <parent link="${parent}"/>
             <child link="wheel_${side}_${part}_link"/>
@@ -53,4 +53,5 @@
             <material>Gazebo/FlatBlack</material>
         </gazebo>
+        <!-- ========================================================== Link -->
     </xacro:macro>
 </robot>
